Commit message: fix DAE file management bug

File: turtlebot_vibot_bringup/urdf/sensors/rplidar.urdf.xacro (robot description, xacro)
@@ -11,5 +11,5 @@
         <origin xyz="0 0 0" rpy="0 0 0"/>
         <geometry>
-            <mesh filename="package://turtlebot_vibot/meshes/sensors/rplidar.dae"/>
+            <mesh filename="package://turtlebot_vibot_bringup/meshes/sensors/rplidar.dae"/>
         </geometry>
       </collision>
@@ -17,5 +17,5 @@
         <origin xyz="0 0 0" rpy="0 0 0"/>
         <geometry>
-            <mesh filename="package://turtlebot_vibot/meshes/sensors/rplidar.dae"/>
+            <mesh filename="package://turtlebot_vibot_bringup/meshes/sensors/rplidar.dae"/>
         </geometry>
       </visual>
